File: CPS_interface.kicad_sch (KiCad schematic)
At the start: 36 parts

Commit message: wip
Parts:
- added U? (x3): TS5A23159DGS, Package_SO:VSSOP-10_3x3mm_P0.5mm, symbol Analog_Switch:TS5A23159DGS
Connections:
- net GND: now also U?.2
- net at R?.2, U?.1: now also U?.9
- net at D?.3: now also U?.10
Other:
- note added: "no bueno"
- moved on the sheet: D?
Changed lines of the file:
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@@
   (junction (at 116.205 175.26) (diameter 0) (color 0 0 0 0)
   )
+  (junction (at 184.15 73.152) (diameter 0) (color 0 0 0 0)
+  )
   (junction (at 132.08 163.83) (diameter 0) (color 0 0 0 0)
   )
@@
     (stroke (width 0) (type default) (color 0 0 0 0))
   )
+  (wire (pts (xy 184.15 73.152) (xy 193.548 73.152))
+    (stroke (width 0) (type default) (color 0 0 0 0))
+  )
   (wire (pts (xy 50.8 76.2) (xy 34.29 76.2))
     (stroke (width 0) (type default) (color 0 0 0 0))
@@
   )
   (wire (pts (xy 115.062 73.66) (xy 124.968 73.66))
+    (stroke (width 0) (type default) (color 0 0 0 0))
+  )
+  (wire (pts (xy 193.548 78.232) (xy 193.548 93.472))
     (stroke (width 0) (type default) (color 0 0 0 0))
   )
@@
     (effects (font (size 1.27 1.27)) (justify left bottom))
   )
+  (text "no bueno " (at 190.246 63.246 0)
+    (effects (font (size 5.08 5.08)) (justify left bottom))
+  )
   (text "400uA=3V" (at 90.17 83.82 0)
     (effects (font (size 1.27 1.27)) (justify left bottom))
@@
     (pin "2")
     (pin "3")
+  )
+  (symbol (lib_id "power:GND") (at 193.548 93.472 0) (unit 1)
+    (in_bom yes) (on_board yes) (fields_autoplaced)
+    (property "Reference" "#PWR?" (id 0) (at 193.548 99.822 0)
+      (effects (font (size 1.27 1.27)) hide)
+    )
+    (property "Value" "GND" (id 1) (at 193.548 98.806 0))
+    (property "Footprint" "" (id 2) (at 193.548 93.472 0)
+      (effects (font (size 1.27 1.27)) hide)
+    )
+    (property "Datasheet" "" (id 3) (at 193.548 93.472 0)
+      (effects (font (size 1.27 1.27)) hide)
+    )
+    (pin "1")
   )
   (symbol (lib_id "power:GND") (at 167.386 146.05 0) (unit 1)
@@
     (pin "1")
   )
+  (symbol (lib_id "Analog_Switch:TS5A23159DGS") (at 226.06 121.92 0) (mirror y) (unit 2)
+    (in_bom yes) (on_board yes) (fields_autoplaced)
+    (property "Reference" "U?" (id 0) (at 226.06 111.76 0))
+    (property "Value" "TS5A23159DGS" (id 1) (at 226.06 114.3 0))
+    (property "Footprint" "Package_SO:VSSOP-10_3x3mm_P0.5mm" (id 2) (at 226.06 125.73 0)
+      (effects (font (size 1.27 1.27)) hide)
+    )
+    (property "Datasheet" "http://www.ti.com/lit/ds/symlink/ts5a23159.pdf" (id 3) (at 252.73 130.81 0)
+      (effects (font (size 1.27 1.27)) hide)
+    )
+    (pin "4")
+    (pin "5")
+    (pin "6")
+    (pin "7")
+  )
   (symbol (lib_id "Diode:1N4148WS") (at 74.93 104.14 0) (mirror y) (unit 1)
     (in_bom yes) (on_board yes) (fields_autoplaced)
@@
     (pin "2")
   )
+  (symbol (lib_id "Analog_Switch:TS5A23159DGS") (at 226.822 149.352 0) (unit 3)
+    (in_bom yes) (on_board yes) (fields_autoplaced)
+    (property "Reference" "U?" (id 0) (at 232.41 148.0819 0)
+      (effects (font (size 1.27 1.27)) (justify left))
+    )
+    (property "Value" "TS5A23159DGS" (id 1) (at 232.41 150.6219 0)
+      (effects (font (size 1.27 1.27)) (justify left))
+    )
+    (property "Footprint" "Package_SO:VSSOP-10_3x3mm_P0.5mm" (id 2) (at 226.822 153.162 0)
+      (effects (font (size 1.27 1.27)) hide)
+    )
+    (property "Datasheet" "http://www.ti.com/lit/ds/symlink/ts5a23159.pdf" (id 3) (at 200.152 158.242 0)
+      (effects (font (size 1.27 1.27)) hide)
+    )
+    (pin "3")
+    (pin "8")
+  )
   (symbol (lib_id "Device:C") (at 74.93 46.99 90) (unit 1)
     (in_bom yes) (on_board yes) (fields_autoplaced)
@@
     (pin "7")
   )
-  (symbol (lib_id "Diode:BAT54S") (at 199.898 82.296 270) (mirror x) (unit 1)
-    (in_bom yes) (on_board yes) (fields_autoplaced)
-    (property "Reference" "D?" (id 0) (at 201.93 81.0259 90)
+  (symbol (lib_id "Diode:BAT54S") (at 213.868 75.692 270) (mirror x) (unit 1)
+    (in_bom yes) (on_board yes) (fields_autoplaced)
+    (property "Reference" "D?" (id 0) (at 215.9 74.4219 90)
       (effects (font (size 1.27 1.27)) (justify left))
     )
-    (property "Value" "BAT54S" (id 1) (at 201.93 83.5659 90)
+    (property "Value" "BAT54S" (id 1) (at 215.9 76.9619 90)
       (effects (font (size 1.27 1.27)) (justify left))
     )
-    (property "Footprint" "Package_TO_SOT_SMD:SOT-23" (id 2) (at 203.073 80.391 0)
+    (property "Footprint" "Package_TO_SOT_SMD:SOT-23" (id 2) (at 217.043 73.787 0)
       (effects (font (size 1.27 1.27)) (justify left) hide)
     )
-    (property "Datasheet" "https://www.diodes.com/assets/Datasheets/ds11005.pdf" (id 3) (at 199.898 85.344 0)
+    (property "Datasheet" "https://www.diodes.com/assets/Datasheets/ds11005.pdf" (id 3) (at 213.868 78.74 0)
       (effects (font (size 1.27 1.27)) hide)
     )
@@
     (pin "3")
   )
+  (symbol (lib_id "Analog_Switch:TS5A23159DGS") (at 201.168 75.692 0) (mirror y) (unit 1)
+    (in_bom yes) (on_board yes) (fields_autoplaced)
+    (property "Reference" "U?" (id 0) (at 201.168 65.278 0))
+    (property "Value" "TS5A23159DGS" (id 1) (at 201.168 67.818 0))
+    (property "Footprint" "Package_SO:VSSOP-10_3x3mm_P0.5mm" (id 2) (at 201.168 79.502 0)
+      (effects (font (size 1.27 1.27)) hide)
+    )
+    (property "Datasheet" "http://www.ti.com/lit/ds/symlink/ts5a23159.pdf" (id 3) (at 227.838 84.582 0)
+      (effects (font (size 1.27 1.27)) hide)
+    )
+    (pin "1")
+    (pin "10")
+    (pin "2")
+    (pin "9")
+  )
   (symbol (lib_id "power:GND") (at 107.188 92.456 0) (unit 1)
