File: HvControl.kicad_sch (KiCad schematic)
At the start: 14 parts

Commit message: wip
Parts:
- added U? (x2): HT7533-1-SOT89, Package_TO_SOT_SMD:SOT-89-3, symbol Regulator_Linear:HT75xx-1-SOT89
Connections:
- net GND: now also U?.1 (GND), U?.1 (GND)
- net at U?.1 (VDD): now also U?.17 (VDD), U?.3 (VOUT)
- net at U?.5 (VDDA): now also U?.3 (VOUT)
Other:
- added sheet CPS interface (CPS_interface.kicad_sch)
- added sheet Gun Interface (Gun_Interface.kicad_sch)

Commit message: wip
Other:
- note added: "optional isolated version: MAX33070E"
Changed lines of the file:
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@@
     (effects (font (size 1.27 1.27)) (justify left bottom))
+  )
+  (text "optional isolated version: MAX33070E  " (at 86.106 144.272 0)
+    (effects (font (size 2.54 2.54)) (justify left bottom))
   )
   (text "need 5V output for isolator" (at 60.96 153.67 0)
@@
       (reference "#PWR?") (unit 1) (value "GND") (footprint "")
     )
+    (path "/168a0226-3f44-46ec-a72a-15290137bd66/2b5dc2db-e1de-4685-af70-bda21c283ac1"
+      (reference "#PWR?") (unit 1) (value "GND") (footprint "")
+    )
     (path "/168a0226-3f44-46ec-a72a-15290137bd66/2dca5777-b212-4811-9d79-1221f2898c3f"
       (reference "#PWR?") (unit 1) (value "GND") (footprint "")
@@
       (reference "U?") (unit 1) (value "MAX14783ExS") (footprint "Package_SO:SOIC-8_3.9x4.9mm_P1.27mm")
     )
+    (path "/168a0226-3f44-46ec-a72a-15290137bd66/c772f9a8-a183-4777-a436-fd70c4943a72"
+      (reference "U?") (unit 1) (value "TS5A23159DGS") (footprint "Package_SO:VSSOP-10_3x3mm_P0.5mm")
+    )
     (path "/168a0226-3f44-46ec-a72a-15290137bd66/d160b7ef-0f83-4fec-8daa-f4a10bee9e0b"
       (reference "U?") (unit 1) (value "TL072") (footprint "")
@@
       (reference "U?") (unit 2) (value "TL072") (footprint "")
     )
+    (path "/168a0226-3f44-46ec-a72a-15290137bd66/950d0cc2-df83-4010-bb7e-8148784ecf71"
+      (reference "U?") (unit 2) (value "TS5A23159DGS") (footprint "Package_SO:VSSOP-10_3x3mm_P0.5mm")
+    )
     (path "/168a0226-3f44-46ec-a72a-15290137bd66/be19c371-58ec-4da8-bf75-bd0c7fa4a358"
       (reference "U?") (unit 2) (value "TL072") (footprint "")
@@
       (reference "U?") (unit 3) (value "TL072") (footprint "")
     )
+    (path "/168a0226-3f44-46ec-a72a-15290137bd66/9f2913ee-f300-41d4-9b7a-339ae5970c4d"
+      (reference "U?") (unit 3) (value "TS5A23159DGS") (footprint "Package_SO:VSSOP-10_3x3mm_P0.5mm")
+    )
     (path "/168a0226-3f44-46ec-a72a-15290137bd66/dfb5e367-b066-4dc5-944f-2f740086ca46"
